Commit message: icra_robot completed

File: robot/urdf/icra_robot.urdf (robot description, URDF)
Before this commit: robot icra_robot, 2 links, 1 joints
Links:
- removed link Untitled
- removed link turret_link
- added link base_link, mass 0.001; collision box size=0.5 0.28033 0.595; visual mesh filename=../meshes/dae/base_link.dae scale=0.001 0.001 0.001
- added link camera_link, mass 0; visual box size=0.04 0.04 0.04
- added link stereo_link, mass 0.001; visual box size=0.16 0.04 0.04
- added link turret_pitch_link, mass 0.001; collision box size=0.10594 0.12283 0.28648; visual mesh filename=../meshes/dae/turret_pitch.dae scale=0.001 0.001 0.001
- added link turret_yaw_link, mass 0.001; collision box size=0.24047 0.21628 0.39979; visual mesh filename=../meshes/dae/turret_yaw.dae scale=0.001 0.001 0.001
Joints:
- removed joint turret_link
- added joint camera_link: type fixed, parent turret_pitch_link, child camera_link, origin xyz=0.15971 0.04459 0.068 rpy=-1.5708 1.5708 0, axis 0 1 0
- added joint stereo_link: type fixed, parent base_link, child stereo_link, origin xyz=0 -0.2 0.07702 rpy=0 0 0, axis 0 1 0
- added joint turret_pitch_joint: type revolute, parent turret_yaw_link, child turret_pitch_link, origin xyz=0.05365 0.02853 0.05461 rpy=1.5708 0 -1.5708, axis 0 0 1.0, limit lower=-1.04 upper=1.04 effort=5.0 velocity=1.0
- added joint turret_yaw_joint: type revolute, parent base_link, child turret_yaw_link, origin xyz=0.01434 -0.02883 0.18781 rpy=0 0 0, axis 0 0 1.0, limit lower=-3.14 upper=3.14 effort=5.0 velocity=1.0
