Commit message: release adjustments

File: urdf/field_no_bounder_no_mesh.urdf (robot description, URDF)
Before this commit: robot unnamed, 14 links, 13 joints
Links:
- link Lfield: geometry 

File: urdf/field_with_mesh.urdf (robot description, URDF)
Before this commit: robot field_with_mesh, 18 links, 17 joints
Links:
- link LA1: geometry collision box size=1.0 0.2 0.4; visual mesh filename=../meshes/dae/A1.dae scale=0.5 0.1 0.2
- link LA2: geometry collision box size=1.0 0.2 0.4; visual mesh filename=../meshes/dae/A2.dae scale=0.5 0.1 0.2
- link LA3: geometry collision box size=1.0 0.2 0.4; visual mesh filename=../meshes/dae/A3.dae scale=0.5 0.1 0.2
- link LA4: geometry collision box size=1.0 0.2 0.4; visual mesh filename=../meshes/dae/A4.dae scale=0.5 0.1 0.2
- link LA5: geometry collision box size=1.0 0.2 0.4; visual mesh filename=../meshes/dae/A5.dae scale=0.5 0.1 0.2
- link LA6: geometry collision box size=1.0 0.2 0.4; visual mesh filename=../meshes/dae/A6.dae scale=0.5 0.1 0.2
- link LB1: geometry collision box size=0.8 0.2 0.4; visual mesh filename=../meshes/dae/B1.dae scale=0.4 0.1 0.2
- link LB2: geometry collision box size=0.8 0.2 0.4; visual mesh filename=../meshes/dae/B2.dae scale=0.4 0.1 0.2
- link LW1: geometry collision box size=0.205 4.89 1.0; visual mesh filename=../meshes/dae/W1.dae scale=0.1025 2.445 0.5
- link LW2: geometry collision box size=0.205 4.89 1.0; visual mesh filename=../meshes/dae/W2.dae scale=0.1025 2.445 0.5
- link LW3: geometry collision box size=8.08 0.205 1.0; visual mesh filename=../meshes/dae/W3.dae scale=4.04 0.1025 0.5
- link LW4: geometry collision box size=8.08 0.205 1.0; visual mesh filename=../meshes/dae/W4.dae scale=4.04 0.1025 0.5
- link Lcenter: geometry collision box size=0.25 0.25 0.4; visual mesh filename=../meshes/dae/center.dae scale=0.125 0.125 0.2

Commit message: fixed field to ground

File: urdf/field_no_bounder_no_mesh.urdf (robot description, URDF)
Before this commit: robot unnamed, 14 links, 13 joints
Links:
- added link world
Joints:
- added joint fixed: type fixed, parent world, child Lfield, origin xyz=0 0 0.5 rpy=0 0 0

File: urdf/field_no_mesh.urdf (robot description, URDF)
Before this commit: robot icra_field, 18 links, 17 joints
Links:
- added link world
Joints:
- added joint fixed: type fixed, parent world, child Lfield, origin xyz=0 0 0.5 rpy=0 0 0

File: urdf/field_with_mesh.urdf (robot description, URDF)
Before this commit: robot field_with_mesh, 18 links, 17 joints
Links:
- added link world
Joints:
- added joint fixed: type fixed, parent world, child Lfield, origin xyz=0 0 0.5 rpy=0 0 0
