Commit message: fix relative path issue by using ROS package path

File: urdf/field_with_mesh.urdf (robot description, URDF)
Before this commit: robot field_with_mesh, 19 links, 18 joints
Links:
- link LA1: geometry collision box size=1.0 0.2 0.4; visual mesh filename=package://irm_icra_simulator/meshes/dae/A1.dae scale=0.5 0.1 0.2
- link LA2: geometry collision box size=1.0 0.2 0.4; visual mesh filename=package://irm_icra_simulator/meshes/dae/A2.dae scale=0.5 0.1 0.2
- link LA3: geometry collision box size=1.0 0.2 0.4; visual mesh filename=package://irm_icra_simulator/meshes/dae/A3.dae scale=0.5 0.1 0.2
- link LA4: geometry collision box size=1.0 0.2 0.4; visual mesh filename=package://irm_icra_simulator/meshes/dae/A4.dae scale=0.5 0.1 0.2
- link LA5: geometry collision box size=1.0 0.2 0.4; visual mesh filename=package://irm_icra_simulator/meshes/dae/A5.dae scale=0.5 0.1 0.2
- link LA6: geometry collision box size=1.0 0.2 0.4; visual mesh filename=package://irm_icra_simulator/meshes/dae/A6.dae scale=0.5 0.1 0.2
- link LB1: geometry collision box size=0.8 0.2 0.4; visual mesh filename=package://irm_icra_simulator/meshes/dae/B1.dae scale=0.4 0.1 0.2
- link LB2: geometry collision box size=0.8 0.2 0.4; visual mesh filename=package://irm_icra_simulator/meshes/dae/B2.dae scale=0.4 0.1 0.2
- link LW1: geometry collision box size=0.205 4.89 1.0; visual mesh filename=package://irm_icra_simulator/meshes/dae/W1.dae scale=0.1025 2.445 0.5
- link LW2: geometry collision box size=0.205 4.89 1.0; visual mesh filename=package://irm_icra_simulator/meshes/dae/W2.dae scale=0.1025 2.445 0.5
- link LW3: geometry collision box size=8.08 0.205 1.0; visual mesh filename=package://irm_icra_simulator/meshes/dae/W3.dae scale=4.04 0.1025 0.5
- link LW4: geometry collision box size=8.08 0.205 1.0; visual mesh filename=package://irm_icra_simulator/meshes/dae/W4.dae scale=4.04 0.1025 0.5
- link Lcenter: geometry collision box size=0.25 0.25 0.4; visual mesh filename=package://irm_icra_simulator/meshes/dae/center.dae scale=0.125 0.125 0.2

File: urdf/icra_robot.urdf (robot description, URDF)
Before this commit: robot icra_robot, 5 links, 4 joints
Links:
- link base_link: geometry collision box size=0.5 0.28033 0.595; visual mesh filename=package://irm_icra_simulator/meshes/dae/base_link.dae scale=0.001 0.001 0.001
- link turret_pitch_link: geometry collision box size=0.10594 0.12283 0.28648; visual mesh filename=package://irm_icra_simulator/meshes/dae/turret_pitch.dae scale=0.001 0.001 0.001
- link turret_yaw_link: geometry collision box size=0.24047 0.21628 0.39979; visual mesh filename=package://irm_icra_simulator/meshes/dae/turret_yaw.dae scale=0.001 0.001 0.001

File: urdf/target_robot.urdf (robot description, URDF)
Before this commit: robot target_robot, 3 links, 2 joints
Links:
- link base_link: geometry collision box size=0.5 0.28033 0.595; visual mesh filename=package://irm_icra_simulator/meshes/dae/base_link.dae scale=0.001 0.001 0.001
- link turret_pitch_link: geometry collision box size=0.10594 0.12283 0.28648; visual mesh filename=package://irm_icra_simulator/meshes/dae/turret_pitch.dae scale=0.001 0.001 0.001
- link turret_yaw_link: geometry collision box size=0.24047 0.21628 0.39979; visual mesh filename=package://irm_icra_simulator/meshes/dae/turret_yaw.dae scale=0.001 0.001 0.001
